File: BC_NFC.kicad_pcb (KiCad board)
At the start: 2 copper layers, 86 x 54 mm, 10 parts, among them U1 NT3H1101W0FHKH

Commit message: Added footprints for NFC chip and antenna.
Parts:
- L1: footprint NFC_antenna:class4_13.56MHz -> footprints:class4_13.56MHz
- R1: value 47R -> 470R
- U1: footprint XQFN8_NT3H1101_NXP:XQFN8_NT3H1101_NXP -> footprints:XQFN8_NT3H1101_NXP
Changed lines of the file:
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@@
     )
   )
-  (footprint "NFC_antenna:class4_13.56MHz" (layer "F.Cu")
+  (footprint "footprints:class4_13.56MHz" (layer "F.Cu")
     (at 184 83.45 90)
     (property "Sheetfile" "BC_NFC.kicad_sch")
@@
         (effects (font (size 1 1) (thickness 0.1)))
     )
-    (fp_text value "2.19uH" (at 0 1 90 unlocked) (layer "F.Fab")
+    (fp_text value "2.19uH" (at 0 1 90 unlocked) (layer "F.Fab") hide
         (effects (font (size 1 1) (thickness 0.15)))
     )
-    (fp_text user "${REFERENCE}" (at 0 2.5 90 unlocked) (layer "F.Fab")
+    (fp_text user "${REFERENCE}" (at 0 2.5 90 unlocked) (layer "F.Fab") hide
         (effects (font (size 1 1) (thickness 0.15)))
     )
@@
     (fp_line (start -20.85 9.55) (end 21.75 9.55)
       (stroke (width 0.3) (type default)) (layer "F.Cu"))
-    (fp_line (start -1.025 -13.05) (end -20.85 -13.05)
+    (fp_line (start -0.825 -13.05) (end -20.85 -13.05)
       (stroke (width 0.3) (type default)) (layer "F.Cu"))
     (fp_line (start 0.05 -13.65) (end -20.85 -13.65)
       (stroke (width 0.3) (type default)) (layer "F.Cu"))
-    (fp_line (start 0.325 -11.875) (end -1.025 -13.05)
+    (fp_line (start 0.325 -11.875) (end -0.825 -13.05)
       (stroke (width 0.3) (type default)) (layer "F.Cu"))
     (fp_line (start 0.4 -14.25) (end -20.85 -14.25)
@@
     (fp_rect (start -24 -18.9) (end 25 10)
       (stroke (width 0.05) (type default)) (fill none) (layer "F.CrtYd"))
+    (dimension (type aligned) (layer "Dwgs.User")
+      (pts (xy 171.1 104.45) (xy 171.1 61.55))
+      (height -11.136426)
+      (gr_text "42.9000 mm" (at 159 83 90) (layer "Dwgs.User")
+        (effects (font (size 1 1) (thickness 0.15)))
+      )
+      (format (prefix "") (suffix "") (units 3) (units_format 1) (precision 4))
+      (style (thickness 0.1) (arrow_length 1.27) (text_position_mode 2) (extension_height 0.58642) (extension_offset 0.5) keep_text_aligned)
+    )
+    (dimension (type aligned) (layer "Dwgs.User")
+      (pts (xy 171.1 61.55) (xy 191 61.55))
+      (height -7.1)
+      (gr_text "19.9000 mm" (at 181.05 53.3) (layer "Dwgs.User")
+        (effects (font (size 1 1) (thickness 0.15)))
+      )
+      (format (prefix "") (suffix "") (units 3) (units_format 1) (precision 4))
+      (style (thickness 0.1) (arrow_length 1.27) (text_position_mode 0) (extension_height 0.58642) (extension_offset 0.5) keep_text_aligned)
+    )
     (dimension (type aligned) (layer "Dwgs.User")
       (pts (xy 168.4 58.85) (xy 193.7 58.85))
@@
       (style (thickness 0.1) (arrow_length 1.27) (text_position_mode 2) (extension_height 0.58642) (extension_offset 0.5) keep_text_aligned)
     )
-    (dimension (type aligned) (layer "Dwgs.User")
-      (pts (xy 171.1 61.55) (xy 191 61.55))
-      (height -7.1)
-      (gr_text "19.9000 mm" (at 181.05 53.3) (layer "Dwgs.User")
-        (effects (font (size 1 1) (thickness 0.15)))
-      )
-      (format (prefix "") (suffix "") (units 3) (units_format 1) (precision 4))
-      (style (thickness 0.1) (arrow_length 1.27) (text_position_mode 0) (extension_height 0.58642) (extension_offset 0.5) keep_text_aligned)
-    )
-    (dimension (type aligned) (layer "Dwgs.User")
-      (pts (xy 171.1 104.45) (xy 171.1 61.55))
-      (height -11.136426)
-      (gr_text "42.9000 mm" (at 159 83 90) (layer "Dwgs.User")
-        (effects (font (size 1 1) (thickness 0.15)))
-      )
-      (format (prefix "") (suffix "") (units 3) (units_format 1) (precision 4))
-      (style (thickness 0.1) (arrow_length 1.27) (text_position_mode 2) (extension_height 0.58642) (extension_offset 0.5) keep_text_aligned)
-    )
     (pad "1" thru_hole circle (at 2.075 -18 90) (size 0.89 0.89) (drill 0.45) (layers "*.Cu")
       (net 4 "Net-(U1-LA)") (pinfunction "1") (pintype "passive"))
@@
       (net 5 "Net-(U1-LB)") (pinfunction "2") (pintype "passive") (zone_connect 2))
     (pad "2" thru_hole circle (at 0.325 -11.875 90) (size 0.89 0.89) (drill 0.45) (layers "*.Cu")
-      (net 5 "Net-(U1-LB)") (pinfunction "2") (pintype "passive") (solder_mask_margin 0.1016) (zone_connect 2))
+      (net 5 "Net-(U1-LB)") (pinfunction "2") (pintype "passive") (zone_connect 2))
   )
   (footprint "Capacitor_SMD:C_0603_1608Metric" (layer "F.Cu")
@@
       (stroke (width 0) (type solid)) (fill solid) (layer "F.SilkS"))
   )
-  (footprint "XQFN8_NT3H1101_NXP:XQFN8_NT3H1101_NXP" (layer "F.Cu")
+  (footprint "footprints:XQFN8_NT3H1101_NXP" (layer "F.Cu")
     (at 137.5757 89.225 90)
     (tags "NT3H1101W0FHKH ")
@@
         (effects (font (size 1 1) (thickness 0.15)))
     )
+    (fp_text user "${REFERENCE}" (at 0 0 90 unlocked) (layer "F.Fab") hide
+        (effects (font (size 1 1) (thickness 0.15)))
+    )
+    (fp_text user "*" (at 0.2667 -0.500126 90) (layer "F.Fab") hide
+        (effects (font (size 1 1) (thickness 0.15)))
+    )
     (fp_text user "*" (at 0.2667 -0.500126 90 unlocked) (layer "F.Fab") hide
         (effects (font (size 1 1) (thickness 0.15)))
     )
-    (fp_text user "*" (at 0.2667 -0.500126 90) (layer "F.Fab") hide
-        (effects (font (size 1 1) (thickness 0.15)))
-    )
-    (fp_text user "${REFERENCE}" (at 0 0 90 unlocked) (layer "F.Fab") hide
-        (effects (font (size 1 1) (thickness 0.15)))
-    )
+    (fp_line (start -0.9525 0.9525) (end -0.43434 0.9525)
+      (stroke (width 0.1524) (type solid)) (layer "F.SilkS"))
+    (fp_line (start -0.43434 -0.9525) (end -0.9525 -0.9525)
+      (stroke (width 0.1524) (type solid)) (layer "F.SilkS"))
+    (fp_line (start 0.43434 0.9525) (end 0.9525 0.9525)
+      (stroke (width 0.1524) (type solid)) (layer "F.SilkS"))
+    (fp_line (start 0.9525 -0.9525) (end 0.43434 -0.9525)
+      (stroke (width 0.1524) (type solid)) (layer "F.SilkS"))
     (fp_line (start -1.3843 -0.855726) (end -1.0795 -0.855726)
       (stroke (width 0.1524) (type solid)) (layer "F.CrtYd"))
@@
     (pad "8" smd rect (at 0 -0.7493 90) (size 0.2032 0.762) (layers "F.Cu" "F.Paste" "F.Mask")
       (net 5 "Net-(U1-LB)") (pinfunction "LB") (pintype "unspecified"))
-    (model "C:/Users/97254/Documents/KiCad/7.0/3dmodels/XQFN8_NT3H1101_NXP.models/XQFN8_NT3H1101_NXP.step"
-      (offset (xyz 0 0 0))
-      (scale (xyz 1 1 1))
-      (rotate (xyz 0 0 0))
-    )
   )
   (footprint "my_logos:Bulb_light" (layer "F.Cu")
@@
         (effects (font (size 1 1) (thickness 0.15)))
     )
-    (fp_text value "47R" (at 0 1.43) (layer "F.Fab") hide
+    (fp_text value "470R" (at 0 1.43) (layer "F.Fab") hide
         (effects (font (size 1 1) (thickness 0.15)))
     )
