File: BC_NFC.kicad_sch (KiCad schematic)
At the start: 5 parts, among them U1 NT3H1101W0FHKH

Commit message: Added footprints for NFC chip and antenna.
Parts:
- L1: footprint NFC_antenna:class4_13.56MHz -> footprints:class4_13.56MHz
- U1: footprint XQFN8_NT3H1101_NXP:XQFN8_NT3H1101_NXP -> footprints:XQFN8_NT3H1101_NXP
Changed lines of the file:
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@@
       (effects (font (face "Segoe UI") (size 2 2) bold))
     )
-    (property "Footprint" "XQFN8_NT3H1101_NXP:XQFN8_NT3H1101_NXP" (at 139.7 68.58 0)
+    (property "Footprint" "footprints:XQFN8_NT3H1101_NXP" (at 139.7 68.58 0)
       (effects (font (size 1.27 1.27) italic) hide)
     )
@@
       (effects (font (face "Segoe UI") (size 2 2) bold))
     )
-    (property "Footprint" "NFC_antenna:class4_13.56MHz" (at 161.29 55.88 0)
+    (property "Footprint" "footprints:class4_13.56MHz" (at 161.29 55.88 0)
       (effects (font (size 1.27 1.27)) hide)
     )
